Commit message: fixed parameter values as written on notion specification.

File: ros2_ws/src/amr_bringup/urdf/amr_robot.urdf.xacro (robot description, xacro)
@@ -90,5 +90,5 @@
   <joint name="lidar_joint" type="fixed">
     <parent link="base_link"/><child link="lidar_link"/>
-    <origin xyz="${lidar_x} 0 ${chassis_height/2.0 + 0.025}" rpy="0 0 0"/>
+    <origin xyz="${lidar_x} 0 ${chassis_height/2.0 + 0.075}" rpy="0 0 0"/>
   </joint>
   <link name="camera_link">
@@ -152,9 +152,9 @@
       <lidar>
         <scan><horizontal>
-          <samples>360</samples><resolution>1</resolution>
+          <samples>720</samples><resolution>1</resolution>
           <min_angle>-3.14159</min_angle><max_angle>3.14159</max_angle>
         </horizontal></scan>
-        <range><min>0.12</min><max>12.0</max><resolution>0.01</resolution></range>
-        <noise><type>gaussian</type><mean>0.0</mean><stddev>0.01</stddev></noise>
+        <range><min>0.12</min><max>25.0</max><resolution>0.01</resolution></range>
+        <noise><type>gaussian</type><mean>0.0</mean><stddev>0.03</stddev></noise>
       </lidar>
     </sensor>

Commit message: fix: [P-4] 카메라 높이 조정 + object_tracker TF 캐싱 최적화

File: ros2_ws/src/amr_bringup/urdf/amr_robot.urdf.xacro (robot description, xacro)
@@ -99,5 +99,5 @@
   <joint name="camera_joint" type="fixed">
     <parent link="base_link"/><child link="camera_link"/>
-    <origin xyz="${camera_x} 0 ${chassis_height/2.0 - 0.05}" rpy="0 0 0"/>
+    <origin xyz="${camera_x} 0 ${chassis_height/2.0 + 0.15}" rpy="0 0 0"/>
   </joint>
   <link name="camera_optical_link"/>
